File: PCB/Lucenox.kicad_pcb (KiCad board)
At the start: 4 copper layers, 348.5 x 118 mm, 253 parts

Commit message: Switch to THT Diodes
Parts:
- D1, D10, D11, D12, D13, D14, D15, D16, D17, D18, D19, D2, D20, D21, D22, D23, D24, D25, D26, D27, D28, D29, D3, D30, D31, D32, D33, D34, D35, D36, D37, D38, D39, D4, D40, D41, D42, D43, D44, D45, D46, D47, D48, D49, D5, D50, D51, D52, D53, D54, D55, D56, D57, D58, D59, D6, D60, D61, D62, D63, D64, D65, D66, D67, D68, D69, D7, D70, D71, D72, D73, D74, D75, D76, D77, D78, D79, D8, D80, D81, D82, D83, D84, D9: footprint Diode_SMD:D_0805_2012Metric -> Diode_THT:D_DO-35_SOD27_P7.62mm_Horizontal
- moved D13 2.47 mm to (328.0, 53.4)
- moved D28 2.47 mm to (351.8, 72.5)
- moved D29 2.47 mm to (370.8, 72.5)
- moved D42 2.47 mm to (280.3, 91.5)
- moved D43 2.47 mm to (299.4, 91.5)
- moved D44 2.47 mm to (323.2, 91.5)
- moved D45 2.47 mm to (351.8, 91.5)
- moved D46 2.47 mm to (370.8, 91.5)
- moved D70 2.47 mm to (256.5, 129.6)
- moved D71 2.47 mm to (275.6, 129.6)
- moved D73 2.47 mm to (370.8, 129.6)
- moved D82 2.47 mm to (351.8, 148.7)
- moved D83 2.47 mm to (370.8, 148.7)
- moved D1 2.47 mm to (61.3, 53.4)
- moved D14 2.47 mm to (61.3, 72.5)
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Routing:
- net ROW4: track 450.3 -> 415.7 mm, vias 17 -> 1
- net GND: track 1893.8 -> 1927.8 mm
- net ROW1: track 354.2 -> 322.8 mm, vias 13 -> 0
- net ROW3: track 425.8 -> 395.8 mm, vias 17 -> 0
- net ROW5: track 399.3 -> 370.9 mm, vias 12 -> 0
- net ROW0: track 353.6 -> 330.6 mm, vias 11 -> 0
- net 5V: track 1810.8 -> 1827.0 mm, vias 17 -> 20
- net ROW2: track 319.1 -> 303.7 mm, vias 13 -> 0
- net RGB: track 157.9 -> 172.8 mm
- net COL5: track 143.2 -> 131.4 mm, vias 2 -> 1
- net RGB_5: track 258.3 -> 269.8 mm
- net COL14: track 264.8 -> 255.7 mm, vias 3 -> 1
- net COL16: track 304.4 -> 312.7 mm
- net COL9: track 207.9 -> 213.9 mm
- net Net-(D43-A): track 8.70 -> 3.31 mm
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