File: PCB/Lucenox.kicad_sch (KiCad schematic)
At the start: 253 parts

Commit message: Switch to THT Diodes
Parts:
- D1, D10, D11, D12, D13, D14, D15, D16, D17, D18, D19, D2, D20, D21, D22, D23, D24, D25, D26, D27, D28, D29, D3, D30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: footprint Diode_SMD:D_0805_2012Metric -> Diode_THT:D_DO-35_SOD27_P7.62mm_Horizontal
